File: ATMega2560/SIM800C.sch (KiCad schematic (older format))
At the start: 39 parts

Commit message: sim800c seperated
Parts:
- added C19: 22pF, Capacitors_SMD:C_0402, symbol C_Small
- added C20: 0.1uF, Capacitors_SMD:C_0402, symbol C_Small
- added C21, C22, C23: 10pF, Capacitors_SMD:C_0402, symbol C_Small
- added C24, C25, C26, C27, C28: 33pF, Capacitors_SMD:C_0402, symbol C_Small
- added C33, C34: DNP, Capacitors_SMD:C_0402, symbol C_Small
- added J28: SIM_Card, symbol SIM_Card
- added J29: 1x8, Pin_Headers:Pin_Header_Straight_1x08_Pitch2.54mm, symbol Conn_01x08
- added J30: SJ-2504A-SMT-TR, symbol SJ-2504A-SMT-TR
- added J32: U.FL, symbol U.FL-R-SMT(10)
- added R10, R11, R12, R13, R14, R15, R16: 1K, Resistors_SMD:R_0402, symbol R_Small
- added R17, R19, R20: 5.6K, Resistors_SMD:R_0402, symbol R_Small
- added R18: 68R, Resistors_SMD:R_0402, symbol R_Small
- added R33: 0R, Resistors_SMD:R_0402, symbol R_Small
- added R7, R8, R9: 51, Resistors_SMD:R_0402, symbol R_Small
- C15, C16, C17, C18, C29, C30, C31, C32: renamed from C?; footprint (none) -> Capacitors_SMD:C_0402
- R21, R22, R23, R24, R25, R26, R27, R28, R29, R30, R31, R32, R34, R35, R36, R37: renamed from R?; footprint (none) -> Resistors_SMD:R_0402
- SW2: renamed from SW?; value SW_Push -> POWER
- U6: renamed from U?; footprint LCC110P1570X1760X250-42N -> (none)
- gave numbers to parts that had none: 13
Connections:
- net labels added: GSM_ANT, MICP, SPKN, SPKP, VCC, Vin
- net labels removed: 12V, VBAT
- wire segments 61 -> 142
- no-connect marks 0 -> 9
Other:
- note added: "4V Buck Converter"
- note added: "Audio Conn"
- note added: "Power Key"
- note added: "SIM Card"
- moved on the sheet: C15, C16, C17, C18, C29, C30, C31, C32, D4, D5, D6, D7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
