File: ATMega2560/ATMega2560.sch (KiCad schematic (older format))
At the start: 73 parts, among them J1 DS18B20, J10 BNC_1, J11 BNC_2, J12 BNC_3, J13 BNC_4, J14 1x8, J15 1x8, J16 1x8, J17 1x8, J18 1x4, J19 1x4, J2 1x3, J20 1x4, J21 1x8, J22 1x2, J23 1x4, J24 1x5, J25 1x3, J26 1x3, J27 1x3, J28 1x3, J29 1x2, J3 1x3, J4 1x3, J5 1x3, J6 1x3, J7 1x3, J8 1x3, J9 1x3, K1 G5Q-1, K2 G5Q-1, K3 G5Q-1, K4 G5Q-1, Q1 2N3055, Q2 2N3055, Q3 2N3055, Q4 2N3055, Q5 SI2323DS, Q6 SI2323DS, SW1 RESET, U1 ATMEGA2560-16AU, U2 DS1302, U3 SN74LVC2T45, U4 LM2574, U5 LM2576, Y1 16Mhz, Y2 32.768 KHz

Commit message: sim800c seperated
Parts:
- removed J15, J17, J21: 1x8, symbol Conn_01x08
- removed Q1, Q2, Q3, Q4: 2N3055, TO_SOT_Packages_THT:TO-3, symbol 2N3055
- added D3, D4, D5, D6: D, symbol D
- added J18: 1x2, Pin_Headers:Pin_Header_Straight_1x02_Pitch2.54mm, symbol Conn_01x02
- added J23: 1x7, Pin_Headers:Pin_Header_Straight_1x07_Pitch2.54mm, symbol Conn_01x07_Female
- added Q1, Q2, Q3, Q4: NMOS, symbol 2N7000
- added R10, R7, R8, R9: 1K, Resistors_SMD:R_0402, symbol R_Small
- added R11, R12, R13, R14: 10K, Resistors_SMD:R_0402, symbol R_Small
- C1: renamed from C4; footprint (none) -> Capacitors_SMD:C_0402_NoSilk
- C10: renamed from C14; footprint (none) -> Capacitors_SMD:C_0402
- C11: renamed from C9; footprint (none) -> Capacitors_SMD:C_0402
- C12: renamed from C13; footprint (none) -> Capacitors_SMD:C_0402
- C13: renamed from C11; footprint (none) -> Capacitors_SMD:C_0402
- C14: renamed from C12; footprint (none) -> Capacitors_SMD:C_0402
- C2: renamed from C1; footprint (none) -> Capacitors_SMD:C_0402
- C3: renamed from C2; footprint (none) -> Capacitors_SMD:C_0402
- C4: renamed from C3; footprint (none) -> Capacitors_SMD:C_0402
- C5, C6: footprint (none) -> Capacitors_SMD:C_0402
- C7: renamed from C10; footprint (none) -> Capacitors_SMD:C_0402
- C8: renamed from C7; footprint (none) -> Capacitors_SMD:C_0402
- C9: renamed from C8; footprint (none) -> Capacitors_SMD:C_0402
- D2: value 1N5822 -> 1N5819; Link (none) -> Value; Manufacturer (none) -> Value; Part Num (none) -> Value; Price (none) -> Value
- J1: renamed from J2; footprint (none) -> Pin_Headers:Pin_Header_Straight_1x03_Pitch2.54mm
- J13: renamed from J18; footprint (none) -> Pin_Headers:Pin_Header_Straight_1x04_Pitch2.54mm
- J14: renamed from J19; footprint (none) -> Pin_Headers:Pin_Header_Straight_1x04_Pitch2.54mm
- J15: renamed from J20; footprint (none) -> Pin_Headers:Pin_Header_Straight_1x04_Pitch2.54mm
- J16: renamed from J14; footprint (none) -> Pin_Headers:Pin_Header_Straight_1x08_Pitch2.54mm
- J17: renamed from J22; footprint (none) -> Pin_Headers:Pin_Header_Straight_1x02_Pitch2.54mm
- J19: renamed from J16; footprint (none) -> Pin_Headers:Pin_Header_Straight_1x08_Pitch2.54mm; Link (none) -> Value; Manufacturer (none) -> Value; Part Num (none) -> Value; Price (none) -> Value
- J2: renamed from J3; footprint (none) -> Pin_Headers:Pin_Header_Straight_1x03_Pitch2.54mm
- J20: renamed from J24; footprint (none) -> Pin_Headers:Pin_Header_Straight_1x05_Pitch2.54mm
- J21: renamed from J23; footprint (none) -> Pin_Headers:Pin_Header_Straight_1x04_Pitch2.54mm
- J22: renamed from J1; value DS18B20 -> 1x3; footprint (none) -> Pin_Headers:Pin_Header_Straight_1x03_Pitch2.54mm
- J24: renamed from J25; footprint (none) -> Pin_Headers:Pin_Header_Straight_1x03_Pitch2.54mm
- J25: renamed from J27; footprint (none) -> Pin_Headers:Pin_Header_Straight_1x03_Pitch2.54mm
- J26: footprint (none) -> Pin_Headers:Pin_Header_Straight_1x03_Pitch2.54mm
- J27: renamed from J28; footprint (none) -> Pin_Headers:Pin_Header_Straight_1x03_Pitch2.54mm
- J28: renamed from J29; footprint (none) -> Pin_Headers:Pin_Header_Straight_1x02_Pitch2.54mm
- J3: renamed from J4; footprint (none) -> Pin_Headers:Pin_Header_Straight_1x03_Pitch2.54mm
- J4: renamed from J5; footprint (none) -> Pin_Headers:Pin_Header_Straight_1x03_Pitch2.54mm
- J5: renamed from J6; footprint (none) -> Pin_Headers:Pin_Header_Straight_1x03_Pitch2.54mm
- J6: renamed from J7; footprint (none) -> Pin_Headers:Pin_Header_Straight_1x03_Pitch2.54mm
- J7: renamed from J8; footprint (none) -> Pin_Headers:Pin_Header_Straight_1x03_Pitch2.54mm
- J8: renamed from J9; footprint (none) -> Pin_Headers:Pin_Header_Straight_1x03_Pitch2.54mm
- Q5: footprint SOT23 -> (none); Field4 Good -> (none); Field5 0.43 USD -> (none); Field6 SOT-23-3 Vishay -> (none); Field7 SI2323DS-T1-GE3 -> (none); Field8 MOSFET P-CH 20V 3.7A SOT23-3 -> (none)
- Q6: footprint SOT23 -> (none); Field4 Good -> (none); Field5 0.43 USD -> (none); Field6 SOT-23-3 Vishay -> (none); Field7 SI2323DS-T1-GE3 -> (none); Field8 MOSFET P-CH 20V 3.7A SOT23-3 -> (none); Manufacturer (none) -> Value
- R1: renamed from R2; footprint (none) -> Resistors_SMD:R_0402
- R2: renamed from R3; footprint (none) -> Resistors_SMD:R_0402
- R3: renamed from R4; footprint (none) -> Resistors_SMD:R_0402
- R4: renamed from R5; footprint (none) -> Resistors_SMD:R_0402
- R5: renamed from R6; footprint (none) -> Resistors_SMD:R_0402
- R6: renamed from R1; footprint (none) -> Resistors_SMD:R_0402
- U2: renamed from U1; footprint TQFP100 -> (none)
- U4: footprint M14B -> (none)
- renumbered D3 to D7, J11 to J10, J12 to J11, J13 to J12, J10 to J9, K2 to K1, K1 to K2, K4 to K3, K3 to K4, U2 to U1
Connections:
- net labels added: PWR_CTRL, PWR_KEY
- net labels removed: RX3, TX3
- wire segments 194 -> 217
Other:
- note added: "RX/TX"
- moved on the sheet: C7, J17, J20, J24, J25, J26, J27, K1, K2, K3, K4

Commit message: BNC, Relay and Regulator connections are made
Parts:
- removed C11: 220uF, Capacitors_SMD:C_0402, symbol C_Small
- removed C7: 0.1uF, Capacitors_SMD:C_0402, symbol C_Small
- removed D2: 1N5819, symbol D_Schottky
- removed D3, D4, D5, D6: D, symbol D
- removed J1, J2, J22, J24, J25, J26, J27, J3, J4, J5, J6, J7, J8: 1x3, Pin_Headers:Pin_Header_Straight_1x03_Pitch2.54mm, symbol Conn_01x03_Female
- removed J10: BNC_2, symbol Conn_Coaxial
- removed J11: BNC_3, symbol Conn_Coaxial
- removed J12: BNC_4, symbol Conn_Coaxial
- removed J13, J14, J15, J21: 1x4, Pin_Headers:Pin_Header_Straight_1x04_Pitch2.54mm, symbol Conn_01x04_Female
- removed J16, J19: 1x8, Pin_Headers:Pin_Header_Straight_1x08_Pitch2.54mm, symbol Conn_01x08
- removed J17: 1x2, Pin_Headers:Pin_Header_Straight_1x02_Pitch2.54mm, symbol Conn_01x02
- removed J20: 1x5, Pin_Headers:Pin_Header_Straight_1x05_Pitch2.54mm, symbol Conn_01x05
- removed J23: 1x7, Pin_Headers:Pin_Header_Straight_1x07_Pitch2.54mm, symbol Conn_01x07_Female
- removed J28: 1x2, Pin_Headers:Pin_Header_Straight_1x02_Pitch2.54mm, symbol Conn_01x02_Female
- removed L1: 330uH, symbol L_Small
- removed Q1, Q2, Q3, Q4: NMOS, symbol 2N7000
- removed Q5, Q6: SI2323DS, symbol SI2323DS-T1-GE3
- removed R10: 1K, Resistors_SMD:R_0402, symbol R_Small
- removed SW1: RESET, symbol SW_Push
- removed U1: DS1302, symbol DS1302
- removed U3: SN74LVC2T45, symbol SN74LVC2T45
- removed U4: LM2574, symbol LM2574
- added BZ1: Buzzer, footprints:MCW12075, symbol Buzzer
- added C15, C16, C17, C2, C20, C21, C25: 0.1uF, Capacitors_SMD:C_0805, symbol C_Small
- added C23: 100uF, Capacitors_SMD:CP_Elec_8x10, symbol CP1_Small
- added C24: 1000uF, Capacitors_SMD:CP_Elec_10x10.5, symbol CP1_Small
- added C26, C27, C28, C29, C3, C30, C31: 1uF, Capacitors_SMD:C_0805, symbol C_Small
- added C32, C33, C34: 2.2uF, Capacitors_SMD:C_0805, symbol C_Small
- added EZ1, EZ2, EZ3, EZ4: EZO-hub, footprints:Atlas_Stamp, symbol EZO-hub
- added J10: TEST_VBat, TestPoint:TestPoint_Pad_D2.0mm, symbol TEST_1P
- added J11: TEST_Reset, TestPoint:TestPoint_Pad_D2.0mm, symbol TEST_1P
- added J12: TEST_MISO, TestPoint:TestPoint_Pad_D2.0mm, symbol TEST_1P
- added J13: TEST_5V, TestPoint:TestPoint_Pad_D2.0mm, symbol TEST_1P
- added J14, J16, J17: BNC_1, footprints:5-1634503-1, symbol Conn_Coaxial
- added J15: BTN, Pin_Headers:Pin_Header_Straight_1x02_Pitch2.54mm, symbol Conn_01x02
- added J18: TEST_MOSI, TestPoint:TestPoint_Pad_D2.0mm, symbol TEST_1P
- added J19: Analog_IN_01x02, footprints:15EDGVC-3.81-02P-14-00AH, symbol Screw_Terminal_01x02
- added J2: Prog_02x04_Odd_Even, Pin_Headers:Pin_Header_Straight_2x04_Pitch1.27mm, symbol Conn_02x04_Odd_Even
- added J20: TEST_3.3V, TestPoint:TestPoint_Pad_D2.0mm, symbol TEST_1P
- added J21: TEST_SCK, TestPoint:TestPoint_Pad_D2.0mm, symbol TEST_1P
- added J22: TEST_GND, TestPoint:TestPoint_Pad_D2.0mm, symbol TEST_1P
- added J23: TEST_RX0, TestPoint:TestPoint_Pad_D2.0mm, symbol TEST_1P
- added J24: TEST_TX0, TestPoint:TestPoint_Pad_D2.0mm, symbol TEST_1P
- added J25: TEST_VDD_EXT, TestPoint:TestPoint_Pad_D2.0mm, symbol TEST_1P
- added J3: Power_IN_01x02, footprints:15EDGVC-3.81-02P-14-00AH, symbol Screw_Terminal_01x02
- added J4: Sensors_02x10_Odd_Even, footprints:DS1013-20SSIB1, symbol Conn_02x10_Odd_Even
- added J5: IO_02x04_Odd_Even, Pin_Headers:Pin_Header_Straight_2x04_Pitch2.54mm, symbol Conn_02x04_Odd_Even
- added J6: I2C, Pin_Headers:Pin_Header_Straight_1x02_Pitch2.54mm, symbol Conn_01x02
- added J7, J8: Screw_Terminal_01x06, footprints:15EGTVC-3.81-06P-14-00AH, symbol Screw_Terminal_01x06
- added Q3, Q4, Q5, Q6: NMOS, TO_SOT_Packages_SMD:SOT-23, symbol Q_NMOS_GSD
- added R11, R18, R22, R28, R3, R30, R31, R4, R7: 4.7K, Resistors_SMD:R_0805, symbol R_Small
- added R15, R16, R25, R27, R29, R32, R33, R34, R35, R36, R38, R6: DNP, Resistors_SMD:R_0805, symbol R_Small
- added R19, R20, R21, R24: 100R, Resistors_SMD:R_0805, symbol R_Small
- added R39, R40, R41: 1K, Resistors_SMD:R_0805, symbol R_Small
- added R42, R43, R44, R45: 10K, Resistors_SMD:R_0805, symbol R_Small
- added R55: 1M, Resistors_SMD:R_0805, symbol R_Small
- added R56: 100K, Resistors_SMD:R_0805, symbol R_Small
- added U1, U10, U6, U9: SI8600, SOIC127P600X175-8N:SOIC127P600X175-8N, symbol SI8600-RESCUE-ATMega2560
- added U11, U12, U14, U5: R1SE-0505, R1SE-0505-R:SOIC254P1110X700-5N, symbol R1SE-0505
- added U15, U16, U17, U8: LD2981ABM, TO_SOT_Packages_SMD:SOT-23-5, symbol LD2981ABM
- added U18: ATMEGA2561-16MU, footprints:ATMEGA2561V-8MU, symbol ATMEGA2561-16MU
- added U19: TXS0102DCUR, TXS0102DCUR:SOP50P310X90-8N, symbol TXS0102DCUR
- added U2: L78L33ABUTR, TO_SOT_Packages_SMD:SOT-89-3, symbol LM2931AZ-5.0_TO92
- added U3: MPCIE-Socket, 2041119-1:TE_2041119-1, symbol MPCIE-Socket
- added U4: DS1302, DS1302ZN_:SOIC127P600X175-8N, symbol DS1302
- BT1: footprint (none) -> footprints:DS1092-04-B6P; Lnk (none) -> Value; MNP (none) -> Value; Price (none) -> Value
- C1: footprint Capacitors_SMD:C_0402_NoSilk -> Capacitors_SMD:C_0805
- C10: renamed from C5; footprint Capacitors_SMD:C_0402 -> Capacitors_SMD:C_0805
- C11: renamed from C6; footprint Capacitors_SMD:C_0402 -> Capacitors_SMD:C_0805
- C12: value 22uF -> 1uF; footprint Capacitors_SMD:C_0402 -> Capacitors_SMD:C_0805
- C13: value 100uF -> 0.1uF; footprint Capacitors_SMD:C_0402 -> Capacitors_SMD:C_0805
- C14: value 1000uF -> 2.2uF; footprint Capacitors_SMD:C_0402 -> Capacitors_SMD:C_0805
- C18: renamed from C10; footprint Capacitors_SMD:C_0402 -> Capacitors_SMD:C_0805
- C5: renamed from C2; footprint Capacitors_SMD:C_0402 -> Capacitors_SMD:C_0805
- C6: renamed from C3; footprint Capacitors_SMD:C_0402 -> Capacitors_SMD:C_0805
- C7: renamed from C4; footprint Capacitors_SMD:C_0402 -> Capacitors_SMD:C_0805
- C8: footprint Capacitors_SMD:C_0402 -> Capacitors_SMD:C_0805
- C9: value 0.1uF -> 0.33uF; footprint Capacitors_SMD:C_0402 -> Capacitors_SMD:C_0805
- D1: footprint (none) -> LEDs:LED_0805
- D3: renamed from D7; value 1N5822 -> 3A-60V; footprint (none) -> Diodes_SMD:D_SMA; Lnk (none) -> Value; MNP (none) -> Value; Price (none) -> Value
- J1: renamed from J18; value 1x2 -> RX/TX
- J9: footprint (none) -> footprints:5-1634503-1; Lnk (none) -> Value; MNP (none) -> Value; Price (none) -> Value
- K1, K2, K3, K4: footprint Relays_THT:Relay_SPDT_OMRON-G5Q -> footprints:HJR-3FF-S-Z-4
- L2: footprint (none) -> footprints:L_SMD_12.5x12.5
- R1, R2: footprint Resistors_SMD:R_0402 -> Resistors_SMD:R_0805
- R10: renamed from R4; Lnk (none) -> Value; MNP (none) -> Value; Price (none) -> Value
- R12, R13: value 10K -> DNP; footprint Resistors_SMD:R_0402 -> Resistors_SMD:R_0805
- R14: value 10K -> 4.7K; footprint Resistors_SMD:R_0402 -> Resistors_SMD:R_0805
- R17: renamed from R5; footprint Resistors_SMD:R_0402 -> Resistors_SMD:R_0805
- R23: renamed from R6; footprint Resistors_SMD:R_0402 -> Resistors_SMD:R_0805
- R26: renamed from R7; footprint Resistors_SMD:R_0402 -> Resistors_SMD:R_0805
- R37: renamed from R11; footprint Resistors_SMD:R_0402 -> Resistors_SMD:R_0805
- R5: renamed from R3; footprint Resistors_SMD:R_0402 -> Resistors_SMD:R_0805
- R8, R9: value 1K -> DNP; footprint Resistors_SMD:R_0402 -> Resistors_SMD:R_0805
- U13: renamed from U5; footprint (none) -> TO_SOT_Packages_SMD:TO-263-5_TabPin3
- U7: renamed from U2; footprint (none) -> ATMEGA2560-16AU:QFP50P1600X1600X120-100N
- Y1: footprint (none) -> CSTCE16M0V53-R0:OSC_CSTCE16M0V53-R0
- Y2: footprint (none) -> footprints:R38-32.768
Connections:
- net labels added: ARD_MISO, ARD_MOSI, ARD_SCK, AREF, BUZZER, GND_ISO1, GND_ISO2, GND_ISO3, GND_ISO4, PIR_DL, PIR_SERIN, PIR_SERIN_REG, PWR_CNTRL, RTC_CE, RTC_MISO, RTC_MOSI, RTC_SCLK, SCREEN_RX, SCREEN_TX, SIM_CLK, SIM_DATA, SIM_RST, SIM_VDD, UART1_CTS, UART1_DCD, UART1_DTR, UART1_RI, UART1_RTS, UART1_RXD, UART1_TXD, US1_ECHO, US1_TR, US2_ECHO, US2_TR, VDD_EXT, VDD_ISO1, VDD_ISO2, VDD_ISO3, VDD_ISO4, XTAL+, XTAL-
- net labels removed: A10, A11, A12, A13, A14, A15, A4, A5, A6, A7, A8, A9, CE, D/L, D22, D23, D24, D29, D42, D43, D44, D45, D46, D47, D48, D49, DIR, EC1, EC2, MISO, MOSI, NX-RX, NX-TX, PWR_CTRL, R1, R2, R3, R4, RX2, SCLK, SERIN, TR1, TR2, TX2
- wire segments 217 -> 404
- no-connect marks 8 -> 57
Other:
- note added: "3.3 LDO"
- note added: "EZO Hubs"
- note added: "Relay Hubs"
- note removed: "+"
- note removed: "-"
- note removed: "5V to 3.3V Buck Conventor"
- note removed: "Analog Pins"
- note removed: "BNC Connectors"
- note removed: "DS18B20"
- note removed: "Digital Pins"
- note removed: "Nextion Screen"
- note removed: "PIR Connection With Level Shifter"
- note removed: "RX/TX Pins"
- note removed: "Relay Outputs"
- note removed: "Relays"
- note removed: "Reverse Current Protection"
- note removed: "TTL Connector"
- note removed: "Ultrasonic Sensors"
- moved on the sheet: BT1, C1, C10, C11, D1, D3, J1, J9, K1, L2, R1, R10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
